File: povDisplay/povDisplayProtoPcb/povDisplayProtoPcb.sch (KiCad schematic (older format))
At the start: 30 parts, among them J0 Conn_01x02

Commit message: Work on pcb.
Parts:
- removed Conn0: Conn_02x06_Counter_Clockwise, symbol Conn_02x06_Counter_Clockwise
- removed Led0, Led1, Led2, Led3, Led4: Conn_02x08_Row_Letter_Last, symbol Conn_02x08_Row_Letter_Last
- removed RNa0, RNa1, RNa2, RNa3, RNb0, RNb1, RNb2, RNb3: R_Network10, Resistors_THT:R_Array_SIP11, symbol R_Network10
- removed Tb1: BUZ11, TO_SOT_Packages_THT:TO-220_Vertical, symbol BUZ11
- added C_Hall0, C_Hall1: C, Capacitors_THT:C_Disc_D7.5mm_W2.5mm_P5.00mm, symbol C
- added Hall_sensor0: Conn_01x03, TO_SOT_Packages_THT:TO-92_Horizontal2_Inline_Narrow_Oval, symbol Conn_01x03
- added J5: Conn_02x06_Odd_Even, Pin_Headers:Pin_Header_Straight_2x06_Pitch2.54mm, symbol Conn_02x06_Odd_Even
- added Led00, Led01, Led10, Led11, Led20, Led21, Led30, Led31, Led40, Led41: Conn_02x04_Odd_Even, Pin_Headers:Pin_Header_Straight_2x04_Pitch2.54mm, symbol Conn_02x04_Odd_Even
- added RNA0, RNA1, RNA2, RNA3, RNA4, RNB0, RNB1, RNB2, RNB3, RNB4: R_Network09, Resistors_THT:R_Array_SIP10, symbol R_Network09
- added R_Hall_0: R, Resistors_THT:R_Axial_DIN0207_L6.3mm_D2.5mm_P7.62mm_Horizontal, symbol R
- added Tb1: BUZ11, TO_SOT_Packages_THT:TO-92_Horizontal2_Inline_Narrow_Oval, symbol IRF4905
- Bat0: renamed from J0; footprint (none) -> Pin_Headers:Pin_Header_Angled_1x02_Pitch2.54mm
- C0, C1, C2, C3, C4, CO0: footprint (none) -> Capacitors_THT:C_Disc_D7.5mm_W2.5mm_P5.00mm
- CI0: footprint (none) -> Capacitors_THT:C_Rect_L4.6mm_W2.0mm_P2.50mm_MKS02_FKP02
- Shift0, Shift1, Shift2, Shift3, Shift4: footprint (none) -> Housings_DIP:DIP-16_W7.62mm_Socket_LongPads
- Ta1: footprint TO_SOT_Packages_THT:TO-220_Vertical -> TO_SOT_Packages_THT:TO-92_Horizontal2_Inline_Narrow_Oval; symbol BUZ11 -> IRF4905
Connections:
- net Clock: now also J5.5 (Pin_5)
- net Command_TA: now also J5.8 (Pin_8)
- net Command_TB: now also J5.10 (Pin_10), Tb1.1 (G)
- net GND: now also C_Hall0.1, C_Hall1.1, Hall_sensor0.3 (Pin_3), J5.1 (Pin_1)
- net Lock: now also J5.3 (Pin_3)
- net Serial_Data_0: now also J5.4 (Pin_4)
- net Serial_Data_1: now also J5.2 (Pin_2)
- net Serial_Data_2: now also J5.7 (Pin_7)
- net Serial_Data_3: now also J5.9 (Pin_9)
- net Serial_Data_4: now also J5.11 (Pin_11)
- net VCC: now also C_Hall0.2, Hall_sensor0.1 (Pin_1), R_Hall_0.2, Tb1.3 (S)
- net at Shift0.1 (QB): now also Led00.3 (Pin_3)
- net at Shift0.15 (QA): now also Led00.1 (Pin_1)
- net at Shift0.2 (QC): now also Led00.5 (Pin_5)
- net at Shift0.3 (QD): now also Led00.7 (Pin_7)
- net at Shift0.4 (QE): now also Led01.1 (Pin_1)
- net at Shift0.5 (QF): now also Led01.3 (Pin_3)
- net at Shift0.6 (QG): now also Led01.5 (Pin_5)
- net at Shift0.7 (QH): now also Led01.7 (Pin_7)
- net at Shift1.1 (QB): now also Led10.3 (Pin_3)
- net at Shift1.15 (QA): now also Led10.1 (Pin_1)
- net at Shift1.2 (QC): now also Led10.5 (Pin_5)
- net at Shift1.3 (QD): now also Led10.7 (Pin_7)
- net at Shift1.4 (QE): now also Led11.1 (Pin_1)
- net at Shift1.5 (QF): now also Led11.3 (Pin_3)
- net at Shift1.6 (QG): now also Led11.5 (Pin_5)
- net at Shift1.7 (QH): now also Led11.7 (Pin_7)
- net at Shift2.1 (QB): now also Led20.3 (Pin_3)
- net at Shift2.15 (QA): now also Led20.1 (Pin_1)
- net at Shift2.2 (QC): now also Led20.5 (Pin_5)
- net at Shift2.3 (QD): now also Led20.7 (Pin_7)
- net at Shift2.4 (QE): now also Led21.1 (Pin_1)
- net at Shift2.5 (QF): now also Led21.3 (Pin_3)
- net at Shift2.6 (QG): now also Led21.5 (Pin_5)
- net at Shift2.7 (QH): now also Led21.7 (Pin_7)
- net at Shift3.1 (QB): now also Led30.3 (Pin_3)
- net at Shift3.15 (QA): now also Led30.1 (Pin_1)
- net at Shift3.2 (QC): now also Led30.5 (Pin_5)
- net at Shift3.3 (QD): now also Led30.7 (Pin_7)
- net at Shift3.4 (QE): now also Led31.1 (Pin_1)
- net at Shift3.5 (QF): now also Led31.3 (Pin_3)
- net at Shift3.6 (QG): now also Led31.5 (Pin_5)
- net at Shift3.7 (QH): now also Led31.7 (Pin_7)
- net at Shift4.1 (QB): now also Led40.3 (Pin_3)
- net at Shift4.15 (QA): now also Led40.1 (Pin_1)
- net at Shift4.2 (QC): now also Led40.5 (Pin_5)
- net at Shift4.3 (QD): now also Led40.7 (Pin_7)
- net at Shift4.4 (QE): now also Led41.1 (Pin_1)
- net at Shift4.5 (QF): now also Led41.3 (Pin_3)
- net at Shift4.6 (QG): now also Led41.5 (Pin_5)
- net at Shift4.7 (QH): now also Led41.7 (Pin_7)
- net Alim_led_1 renamed Alim_led_A
- net Alim_led_A: now also RNA0.1 (common), RNA1.1 (common), RNA2.1 (common), RNA3.1 (common), RNA4.1 (common)
- new net: Led00.2 (Pin_2), RNA0.10 (R9), RNB0.10 (R9)
- new net: Led10.2 (Pin_2), RNA0.2 (R1), RNB0.2 (R1)
- new net: Led01.8 (Pin_8), RNA0.3 (R2), RNB0.3 (R2)
- new net: Led01.6 (Pin_6), RNA0.4 (R3), RNB0.4 (R3)
- new net: Led01.4 (Pin_4), RNA0.5 (R4), RNB0.5 (R4)
- new net: Led01.2 (Pin_2), RNA0.6 (R5), RNB0.6 (R5)
- new net: Led00.8 (Pin_8), RNA0.7 (R6), RNB0.7 (R6)
- new net: Led00.6 (Pin_6), RNA0.8 (R7), RNB0.8 (R7)
- new net: Led00.4 (Pin_4), RNA0.9 (R8), RNB0.9 (R8)
- new net: Led20.4 (Pin_4), RNA1.10 (R9), RNB1.10 (R9)
- new net: Led10.4 (Pin_4), RNA1.2 (R1), RNB1.2 (R1)
- new net: Led10.6 (Pin_6), RNA1.3 (R2), RNB1.3 (R2)
- new net: Led10.8 (Pin_8), RNA1.4 (R3), RNB1.4 (R3)
- new net: Led11.2 (Pin_2), RNA1.5 (R4), RNB1.5 (R4)
- new net: Led11.4 (Pin_4), RNA1.6 (R5), RNB1.6 (R5)
- new net: Led11.6 (Pin_6), RNA1.7 (R6), RNB1.7 (R6)
- new net: Led11.8 (Pin_8), RNA1.8 (R7), RNB1.8 (R7)
- new net: Led20.2 (Pin_2), RNA1.9 (R8), RNB1.9 (R8)
- new net: Led20.6 (Pin_6), RNA2.10 (R9), RNB2.10 (R9)
- new net: Led30.6 (Pin_6), RNA2.2 (R1), RNB2.2 (R1)
- new net: Led30.4 (Pin_4), RNA2.3 (R2), RNB2.3 (R2)
- new net: Led30.2 (Pin_2), RNA2.4 (R3), RNB2.4 (R3)
- new net: Led21.8 (Pin_8), RNA2.5 (R4), RNB2.5 (R4)
- new net: Led21.6 (Pin_6), RNA2.6 (R5), RNB2.6 (R5)
- new net: Led21.4 (Pin_4), RNA2.7 (R6), RNB2.7 (R6)
- new net: Led21.2 (Pin_2), RNA2.8 (R7), RNB2.8 (R7)
- new net: Led20.8 (Pin_8), RNA2.9 (R8), RNB2.9 (R8)
- new net: Led40.8 (Pin_8), RNA3.10 (R9), RNB3.10 (R9)
- new net: Led30.8 (Pin_8), RNA3.2 (R1), RNB3.2 (R1)
- new net: Led31.2 (Pin_2), RNA3.3 (R2), RNB3.3 (R2)
- new net: Led31.4 (Pin_4), RNA3.4 (R3), RNB3.4 (R3)
- new net: Led31.6 (Pin_6), RNA3.5 (R4), RNB3.5 (R4)
- new net: Led31.8 (Pin_8), RNA3.6 (R5), RNB3.6 (R5)
- new net: Led40.2 (Pin_2), RNA3.7 (R6), RNB3.7 (R6)
- new net: Led40.4 (Pin_4), RNA3.8 (R7), RNB3.8 (R7)
- new net: Led40.6 (Pin_6), RNA3.9 (R8), RNB3.9 (R8)
- new net: Led41.8 (Pin_8), RNA4.5 (R4), RNB4.5 (R4)
- new net: Led41.6 (Pin_6), RNA4.6 (R5), RNB4.6 (R5)
- new net: Led41.4 (Pin_4), RNA4.7 (R6), RNB4.7 (R6)
- new net: Led41.2 (Pin_2), RNA4.8 (R7), RNB4.8 (R7)
- new net Alime_led_B: RNB0.1 (common), RNB1.1 (common), RNB2.1 (common), RNB3.1 (common), RNB4.1 (common), Tb1.2 (D)
- new net Hall_Sensor: C_Hall1.2, Hall_sensor0.2 (Pin_2), J5.12 (Pin_12), R_Hall_0.1
- no-connect marks 7 -> 16
Other:
- moved on the sheet: Bat0, Shift0, Shift1, Shift2, Shift3, Shift4
