File: povDisplay/povDisplayProtoPcb/povDisplayProtoPcb3.kicad_pcb (KiCad board)
At the start: 4 copper layers, 41 parts, among them J5 Conn_02x06_Odd_Even

Commit message: Work on pcb.
Parts:
- Bat0: moved to F.Cu
- moved Bat0 73.7 mm to (109.9, 31.8), turned to 0 degrees
- moved LM7805 55.9 mm to (127.6, 24.8), turned to 0 degrees
- moved CI0 54.8 mm to (127.6, 38.1)
- moved C_Hall1 54.7 mm to (135.3, 32.4), turned to 0 degrees
- moved CO0 36.6 mm to (150.5, 25.4)
- moved J5 25.5 mm to (161.3, 110.5)
- moved C1 19.9 mm to (181.0, 122.6)
- moved R_Hall_0 19.4 mm to (185.4, 47.6), turned to 270 degrees
- moved Shift1 19.4 mm to (187.3, 119.4)
- moved C3 15.3 mm to (181.0, 81.9)
- moved Shift3 14.7 mm to (187.3, 78.7)
- moved Ta1 9.16 mm to (195.6, 31.8)
- moved Tb1 8.03 mm to (182.9, 31.8)
- moved C2 7.02 mm to (195.6, 102.2)
- moved RNB4 6.99 mm to (225.4, 28.6)
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Connections:
- RNA4 pad 10: Net-(RNA4-Pad10) -> Net-(Led41-Pad2)
- RNA4 pad 5: Net-(Led41-Pad8) -> Net-(RNA4-Pad5)
- RNA4 pad 6: Net-(Led41-Pad6) -> Net-(RNA4-Pad6)
- RNA4 pad 7: Net-(Led41-Pad4) -> Net-(Led41-Pad8)
- RNA4 pad 8: Net-(Led41-Pad2) -> Net-(Led41-Pad6)
- RNA4 pad 9: Net-(RNA4-Pad9) -> Net-(Led41-Pad4)
- RNB4 pad 10: Net-(RNB4-Pad10) -> Net-(Led41-Pad2)
- RNB4 pad 5: Net-(Led41-Pad8) -> Net-(RNB4-Pad5)
- RNB4 pad 6: Net-(Led41-Pad6) -> Net-(RNB4-Pad6)
- RNB4 pad 7: Net-(Led41-Pad4) -> Net-(Led41-Pad8)
- RNB4 pad 8: Net-(Led41-Pad2) -> Net-(Led41-Pad6)
- RNB4 pad 9: Net-(RNB4-Pad9) -> Net-(Led41-Pad4)
Routing:
- net GND: track 242.4 -> 20.9 mm
- net VCC: track 224.0 -> 26.7 mm, vias 10 -> 2
- net Alime_led_B: track 249.3 -> 77.1 mm
- net Clock: track 156.3 -> 0.00 mm, vias 8 -> 0
- net Lock: track 145.8 -> 0.00 mm, vias 4 -> 0
- net Alim_led_A: track 165.9 -> 25.0 mm, vias 4 -> 3
- net Command_TA: track 135.8 -> 0.00 mm, vias 4 -> 0
- net Hall_Sensor: track 116.5 -> 0.00 mm, vias 2 -> 0
- net Command_TB: track 94.9 -> 0.00 mm
- net Serial_Data_4: track 81.2 -> 0.00 mm
- net Serial_Data_3: track 50.6 -> 0.00 mm, vias 2 -> 0
- net Serial_Data_0: track 42.8 -> 0.00 mm
- net Serial_Data_2: track 28.5 -> 0.00 mm, vias 2 -> 0
- net Net-(Led10-Pad1): track 27.8 -> 0.00 mm, vias 2 -> 0
- net Net-(Led20-Pad1): track 26.4 -> 0.00 mm, vias 2 -> 0
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