File: povDisplay/povDisplayProtoPcb/povDisplayProtoPcb4.kicad_pcb (KiCad board)
At the start: 4 copper layers, 41 parts, among them J5 Conn_02x06_Odd_Even

Commit message: Work on pcb.
Parts:
- Bat0: moved to F.Cu
- moved Bat0 73.7 mm to (109.9, 31.8), turned to 0 degrees
- moved J5 25.5 mm to (161.3, 110.5)
- moved RNB4 6.99 mm to (225.4, 28.6)
- moved Led41 0.64 mm to (207.0, 47.0)
- moved C_Hall1 0.63 mm to (190.5, 36.1)
Connections:
- RNA4 pad 10: Net-(RNA4-Pad10) -> Net-(Led41-Pad2)
- RNA4 pad 5: Net-(Led41-Pad8) -> Net-(RNA4-Pad5)
- RNA4 pad 6: Net-(Led41-Pad6) -> Net-(RNA4-Pad6)
- RNA4 pad 7: Net-(Led41-Pad4) -> Net-(Led41-Pad8)
- RNA4 pad 8: Net-(Led41-Pad2) -> Net-(Led41-Pad6)
- RNA4 pad 9: Net-(RNA4-Pad9) -> Net-(Led41-Pad4)
- RNB4 pad 10: Net-(RNB4-Pad10) -> Net-(Led41-Pad2)
- RNB4 pad 5: Net-(Led41-Pad8) -> Net-(RNB4-Pad5)
- RNB4 pad 6: Net-(Led41-Pad6) -> Net-(RNB4-Pad6)
- RNB4 pad 7: Net-(Led41-Pad4) -> Net-(Led41-Pad8)
- RNB4 pad 8: Net-(Led41-Pad2) -> Net-(Led41-Pad6)
- RNB4 pad 9: Net-(RNB4-Pad9) -> Net-(Led41-Pad4)
Routing:
- net Clock: track 156.3 -> 4.44 mm, vias 8 -> 1
- net Lock: track 145.8 -> 2.54 mm, vias 4 -> 1
- net Alime_led_B: track 249.3 -> 112.3 mm
- net Command_TA: track 135.8 -> 3.81 mm, vias 4 -> 1
- net Alim_led_A: track 165.9 -> 42.5 mm, vias 4 -> 3
- net Hall_Sensor: track 116.5 -> 24.1 mm, vias 2 -> 0
- net Serial_Data_4: track 81.2 -> 0.00 mm
- net Command_TB: track 94.9 -> 35.9 mm
- net Serial_Data_3: track 50.6 -> 0.00 mm, vias 2 -> 0
- net Serial_Data_0: track 42.8 -> 0.00 mm
- net GND: track 242.4 -> 206.9 mm
- net Serial_Data_2: track 28.5 -> 0.00 mm, vias 2 -> 0
- net Serial_Data_1: track 19.1 -> 0.00 mm, vias 2 -> 0
- net Net-(Led41-Pad8): track 8.89 -> 0.00 mm
- net Net-(Led41-Pad6): track 8.89 -> 0.00 mm
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