File: povDisplay/povDisplayProtoPcb/povDisplayProtoPcb6.kicad_pcb (KiCad board)
At the start: 4 copper layers, 41 parts, among them J5 Conn_02x06_Odd_Even

Commit message: Work on pcb.
Routing:
- net GND: track 242.4 -> 243.2 mm
- net Hall_Sensor: track 116.5 -> 117.2 mm
Changed lines of the file:
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@@
     (thickness 1.6)
     (drawings 0)
-    (tracks 706)
+    (tracks 704)
     (zones 0)
     (modules 41)
@@
   )
   (setup
-    (last_trace_width 1)
+    (last_trace_width 1.6)
     (user_trace_width 0.6)
     (user_trace_width 1)
@@
     (mod_text_size 1 1)
     (mod_text_width 0.15)
-    (pad_size 1.9 1.9)
-    (pad_drill 1)
+    (pad_size 1.524 1.524)
+    (pad_drill 0.762)
     (pad_to_mask_clearance 0.2)
     (aux_axis_origin 0 0)
@@
     (pad 1 thru_hole rect (at 0 0 90) (size 1.8 1.8) (drill 1) (layers *.Cu *.Mask)
       (net 1 Vbat))
-    (pad 2 thru_hole oval (at 2.54 0 90) (size 1.6 1.8) (drill 1) (layers *.Cu *.Mask)
+    (pad 2 thru_hole oval (at 2.54 0 90) (size 1.8 1.8) (drill 1) (layers *.Cu *.Mask)
       (net 2 GND))
-    (pad 3 thru_hole oval (at 5.08 0 90) (size 1.6 1.8) (drill 1) (layers *.Cu *.Mask)
+    (pad 3 thru_hole oval (at 5.08 0 90) (size 1.8 1.8) (drill 1) (layers *.Cu *.Mask)
       (net 3 VCC))
     (model ${KISYS3DMOD}/TO_SOT_Packages_THT.3dshapes/TO-220_Vertical.wrl
@@
     (pad 1 thru_hole rect (at 0 0) (size 1.8 1.8) (drill 1) (layers *.Cu *.Mask)
       (net 10 Command_TA))
-    (pad 2 thru_hole oval (at 2.54 0) (size 1.6 1.8) (drill 1) (layers *.Cu *.Mask)
+    (pad 2 thru_hole oval (at 2.54 0) (size 1.8 1.8) (drill 1) (layers *.Cu *.Mask)
       (net 13 Alim_led_A))
-    (pad 3 thru_hole oval (at 5.08 0) (size 1.6 1.8) (drill 1) (layers *.Cu *.Mask)
+    (pad 3 thru_hole oval (at 5.08 0) (size 1.8 1.8) (drill 1) (layers *.Cu *.Mask)
       (net 3 VCC))
     (model ${KISYS3DMOD}/TO_SOT_Packages_THT.3dshapes/TO-220_Vertical.wrl
@@
     (pad 1 thru_hole rect (at 0 0) (size 1.8 1.8) (drill 1) (layers *.Cu *.Mask)
       (net 9 Command_TB))
-    (pad 2 thru_hole oval (at 2.54 0) (size 1.6 1.8) (drill 1) (layers *.Cu *.Mask)
+    (pad 2 thru_hole oval (at 2.54 0) (size 1.8 1.8) (drill 1) (layers *.Cu *.Mask)
       (net 14 Alime_led_B))
-    (pad 3 thru_hole oval (at 5.08 0) (size 1.6 1.8) (drill 1) (layers *.Cu *.Mask)
+    (pad 3 thru_hole oval (at 5.08 0) (size 1.8 1.8) (drill 1) (layers *.Cu *.Mask)
       (net 3 VCC))
     (model ${KISYS3DMOD}/TO_SOT_Packages_THT.3dshapes/TO-220_Vertical.wrl
@@
       (effects (font (size 1 1) (thickness 0.15)))
     )
-    (pad 1 thru_hole circle (at 0 0 90) (size 1.9 1.9) (drill 1) (layers *.Cu *.Mask)
+    (pad 1 thru_hole circle (at 0 0 90) (size 2 2) (drill 1) (layers *.Cu *.Mask)
       (net 2 GND))
     (pad 2 thru_hole circle (at 5 0 90) (size 2 2) (drill 1) (layers *.Cu *.Mask)
@@
     (pad 1 thru_hole rect (at 0 0) (size 1.8 1.8) (drill 1) (layers *.Cu *.Mask)
       (net 3 VCC))
-    (pad 2 thru_hole oval (at 2.54 0) (size 1.6 1.8) (drill 1) (layers *.Cu *.Mask)
+    (pad 2 thru_hole oval (at 2.54 0) (size 1.8 1.8) (drill 1) (layers *.Cu *.Mask)
       (net 26 Hall_Sensor))
     (pad 3 thru_hole oval (at 5.08 0) (size 1.8 1.8) (drill 1) (layers *.Cu *.Mask)
@@
   (segment (start 182.245 36.83) (end 182.245 41.87) (width 1.6) (layer F.Cu) (net 1))
   (segment (start 182.245 41.87) (end 182.285 41.91) (width 1.6) (layer F.Cu) (net 1))
-  (segment (start 201.93 36.195) (end 203.680399 36.195) (width 1) (layer F.Cu) (net 2))
-  (segment (start 203.680399 36.195) (end 204.061399 36.576) (width 1) (layer F.Cu) (net 2))
-  (segment (start 204.061399 36.576) (end 208.026 36.576) (width 1) (layer F.Cu) (net 2))
-  (segment (start 201.93 36.195) (end 201.93 36.068) (width 1) (layer F.Cu) (net 2))
-  (segment (start 201.93 36.068) (end 202.438 36.576) (width 1) (layer F.Cu) (net 2))
-  (segment (start 208.026 36.576) (end 210.82 33.782) (width 1) (layer F.Cu) (net 2))
-  (segment (start 210.82 33.782) (end 210.82 32.385) (width 1) (layer F.Cu) (net 2))
   (segment (start 194.31 72.39) (end 199.12999 72.39) (width 1.6) (layer F.Cu) (net 2))
   (segment (start 199.12999 98.425) (end 199.22999 98.425) (width 1.4) (layer F.Cu) (net 2))
@@
   (segment (start 184.865 34.29) (end 186.69 36.115) (width 1.6) (layer F.Cu) (net 2))
   (segment (start 210.82 29.845) (end 210.82 32.385) (width 1.6) (layer F.Cu) (net 2))
+  (segment (start 210.82 32.385) (end 210.82 36.195) (width 1) (layer F.Cu) (net 2))
+  (segment (start 201.93 36.195) (end 202.36999 36.63499) (width 1) (layer F.Cu) (net 2))
+  (segment (start 202.36999 36.63499) (end 203.199852 36.63499) (width 1) (layer F.Cu) (net 2))
+  (segment (start 203.199852 36.63499) (end 203.394862 36.83) (width 1) (layer F.Cu) (net 2))
+  (segment (start 203.394862 36.83) (end 210.185 36.83) (width 1) (layer F.Cu) (net 2))
+  (segment (start 210.185 36.83) (end 210.82 36.195) (width 1) (layer F.Cu) (net 2))
   (segment (start 200.025 36.195) (end 199.22999 36.99001) (width 1.4) (layer F.Cu) (net 2))
   (segment (start 201.93 36.195) (end 200.025 36.195) (width 1.4) (layer F.Cu) (net 2))
@@
   (via (at 189.865 121.92) (size 1.4) (drill 0.4) (layers F.Cu B.Cu) (net 11))
   (segment (start 191.77 43.815) (end 191.77 69.85) (width 0.6) (layer B.Cu) (net 11))
-  (via (at 191.77 69.85) (size 1.4) (drill 0.4) (layers F.Cu B.Cu) (net 11))
+  (via (at 191.77 69.85) (size 1.4) (drill 0.4) (layers F.Cu B.Cu) (net 11) (status 1000000))
   (segment (start 194.31 43.815) (end 191.77 43.815) (width 1) (layer F.Cu) (net 11))
   (via (at 191.77 43.815) (size 1.4) (drill 0.4) (layers F.Cu B.Cu) (net 11))
@@
   (segment (start 218.44 133.985) (end 218.44 135.19499) (width 1.8) (layer F.Cu) (net 14))
   (segment (start 218.44 132.715) (end 218.44 133.985) (width 1.8) (layer F.Cu) (net 14))
-  (segment (start 208.28 31.745) (end 208.28 29.845) (width 1) (layer F.Cu) (net 26))
-  (segment (start 208.28 33.329002) (end 208.28 31.745) (width 1) (layer F.Cu) (net 26))
-  (segment (start 204.715999 34.685001) (end 206.924001 34.685001) (width 1) (layer F.Cu) (net 26))
-  (segment (start 196.420136 31.115) (end 198.325136 33.02) (width 1) (layer F.Cu) (net 26))
-  (segment (start 195.58 31.115) (end 196.420136 31.115) (width 1) (layer F.Cu) (net 26))
-  (segment (start 198.325136 33.02) (end 203.050998 33.02) (width 1) (layer F.Cu) (net 26))
-  (segment (start 203.050998 33.02) (end 204.715999 34.685001) (width 1) (layer F.Cu) (net 26))
-  (segment (start 206.924001 34.685001) (end 208.28 33.329002) (width 1) (layer F.Cu) (net 26))
   (segment (start 189.865 31.115) (end 195.58 31.115) (width 1.6) (layer F.Cu) (net 26))
   (segment (start 180.086 68.58) (end 180.086 110.744) (width 1) (layer F.Cu) (net 26))
@@
   (segment (start 190.5 31.115) (end 192.786 31.115) (width 1) (layer F.Cu) (net 26))
   (via (at 192.786 31.115) (size 1.4) (drill 0.4) (layers F.Cu B.Cu) (net 26))
+  (segment (start 195.58 31.115) (end 196.420136 31.115) (width 1) (layer F.Cu) (net 26))
+  (segment (start 196.420136 31.115) (end 198.325136 33.02) (width 1) (layer F.Cu) (net 26))
+  (segment (start 198.325136 33.02) (end 202.124862 33.02) (width 1) (layer F.Cu) (net 26))
+  (segment (start 202.124862 33.02) (end 204.029862 34.925) (width 1) (layer F.Cu) (net 26))
+  (segment (start 204.029862 34.925) (end 207.645 34.925) (width 1) (layer F.Cu) (net 26))
+  (segment (start 207.645 34.925) (end 208.28 34.29) (width 1) (layer F.Cu) (net 26))
+  (segment (start 208.28 34.29) (end 208.28 31.117792) (width 1) (layer F.Cu) (net 26))
+  (segment (start 208.28 31.117792) (end 208.28 29.845) (width 1) (layer F.Cu) (net 26))
   (segment (start 194.31 155.575) (end 198.755 155.575) (width 1) (layer F.Cu) (net 27))
   (segment (start 198.755 155.575) (end 199.39 156.21) (width 1) (layer F.Cu) (net 27))
@@
   (segment (start 201.93 48.895) (end 204.13 48.895) (width 1) (layer F.Cu) (net 97))
   (segment (start 204.13 48.895) (end 204.765 49.53) (width 1) (layer F.Cu) (net 97))
-  (segment (start 209.55 51.435) (end 211.455 51.435) (width 1) (layer F.Cu) (net 98))
-  (segment (start 213.995 53.975) (end 214.63 53.975) (width 1) (layer F.Cu) (net 98))
-  (segment (start 211.455 51.435) (end 213.995 53.975) (width 1) (layer F.Cu) (net 98))
+  (segment (start 209.55 51.435) (end 212.09 51.435) (width 1) (layer F.Cu) (net 98))
+  (segment (start 212.09 51.435) (end 214.63 53.975) (width 1) (layer F.Cu) (net 98))
   (segment (start 214.63 53.975) (end 218.44 53.975) (width 1.6) (layer F.Cu) (net 98))
   (segment (start 201.93 46.355) (end 207.01 46.355) (width 1) (layer F.Cu) (net 99))
