File: povDisplay/povDisplayProtoPcb/_autosave-povDisplayProtoPcb.kicad_pcb (KiCad board)
At the start: 4 copper layers, 41 parts, among them J5 Conn_02x06_Odd_Even

Commit message: Add cutting edge.
Other:
- board outline added: 49.3 x 149.1 mm
Changed lines of the file:
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@@
     (links 195)
     (no_connects 0)
-    (area 0 0 0 0)
+    (area 170.869999 7.69 224.103001 164.667001)
     (thickness 1.6)
-    (drawings 0)
+    (drawings 11)
     (tracks 706)
     (zones 0)
@@
     (pad_drill 1)
     (pad_to_mask_clearance 0.2)
-    (aux_axis_origin 176.276 16.764)
+    (aux_axis_origin 174.752 15.494)
     (visible_elements FFFFEF7F)
     (pcbplotparams
-      (layerselection 0x00000_80000000)
+      (layerselection 0x01000_80000000)
       (usegerberextensions false)
       (excludeedgelayer true)
@@
     )
   )
+  (gr_line (start 174.752 164.592) (end 177.038 164.592) (angle 90) (layer Edge.Cuts) (width 0.15))
+  (gr_line (start 174.752 163.83) (end 174.752 164.592) (angle 90) (layer Edge.Cuts) (width 0.15))
+  (gr_line (start 224.028 164.592) (end 224.028 163.83) (angle 90) (layer Edge.Cuts) (width 0.15))
+  (gr_line (start 222.504 164.592) (end 224.028 164.592) (angle 90) (layer Edge.Cuts) (width 0.15))
+  (gr_line (start 224.028 15.494) (end 224.028 16.764) (angle 90) (layer Edge.Cuts) (width 0.15))
+  (gr_line (start 220.98 15.494) (end 224.028 15.494) (angle 90) (layer Edge.Cuts) (width 0.15))
+  (gr_line (start 174.752 15.494) (end 174.752 16.764) (angle 90) (layer Edge.Cuts) (width 0.15))
+  (gr_line (start 174.752 163.83) (end 174.752 16.764) (angle 90) (layer Edge.Cuts) (width 0.15))
+  (gr_line (start 222.504 164.592) (end 176.784 164.592) (angle 90) (layer Edge.Cuts) (width 0.15))
+  (gr_line (start 224.028 16.764) (end 224.028 163.83) (angle 90) (layer Edge.Cuts) (width 0.15))
+  (gr_line (start 174.752 15.494) (end 220.98 15.494) (angle 90) (layer Edge.Cuts) (width 0.15))
   (segment (start 182.285 41.91) (end 182.285 45.68) (width 1.6) (layer B.Cu) (net 1))
   (segment (start 182.285 45.68) (end 182.245 45.72) (width 1.6) (layer B.Cu) (net 1))
